File: PCB_Files/BarLight_v1.kicad_sch (KiCad schematic)
At the start: 2 parts, among them U1 ATtiny85-20P, U2 LF50_TO220

Commit message: added reset switch to project schematic
Parts:
- added SW1: SW_Push, symbol Switch:SW_Push
Connections:
- net GND: now also SW1.2
- net at U1.1 (~{RESET}/PB5): now also SW1.1
Changed lines of the file:
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@@
+    (stroke (width 0) (type default))
+  )
+  (wire (pts (xy 137.16 95.25) (xy 138.43 95.25))
+    (stroke (width 0) (type default))
+  )
+  (wire (pts (xy 148.59 95.25) (xy 149.86 95.25))
     (stroke (width 0) (type default))
   )
   (wire (pts (xy 129.54 30.48) (xy 128.27 30.48))
+    (stroke (width 0) (type default))
+  )
+  (wire (pts (xy 137.16 86.36) (xy 137.16 95.25))
+    (stroke (width 0) (type default))
+  )
+  (wire (pts (xy 135.89 86.36) (xy 137.16 86.36))
+    (stroke (width 0) (type default))
+  )
+  (wire (pts (xy 149.86 95.25) (xy 149.86 96.52))
     (stroke (width 0) (type default))
   )
@@
         (path "/e09a2a5b-1bf6-492a-87e7-b4fbc0e9cc1e"
           (reference "#PWR05") (unit 1)
+        )
+      )
+    )
+  )
+  (symbol (lib_id "power:GND") (at 149.86 96.52 0) (unit 1)
+    (in_bom yes) (on_board yes) (dnp no) (fields_autoplaced)
+    (property "Reference" "#PWR06" (at 149.86 102.87 0)
+      (effects (font (size 1.27 1.27)) hide)
+    )
+    (property "Value" "GND" (at 149.86 101.6 0)
+      (effects (font (size 1.27 1.27)))
+    )
+    (property "Footprint" "" (at 149.86 96.52 0)
+      (effects (font (size 1.27 1.27)) hide)
+    )
+    (property "Datasheet" "" (at 149.86 96.52 0)
+      (effects (font (size 1.27 1.27)) hide)
+    )
+    (pin "1")
+    (instances
+      (project "BarLight_v1"
+        (path "/e09a2a5b-1bf6-492a-87e7-b4fbc0e9cc1e"
+          (reference "#PWR06") (unit 1)
         )
       )
@@
         )
       )
+    )
+  )
+  (symbol (lib_id "Switch:SW_Push") (at 143.51 95.25 0) (unit 1)
+    (in_bom yes) (on_board yes) (dnp no) (fields_autoplaced)
+    (property "Reference" "SW1" (at 143.51 88.9 0)
+      (effects (font (size 1.27 1.27)))
+    )
+    (property "Value" "SW_Push" (at 143.51 91.44 0)
+      (effects (font (size 1.27 1.27)))
+    )
+    (property "Footprint" "" (at 143.51 90.17 0)
+      (effects (font (size 1.27 1.27)) hide)
+    )
+    (property "Datasheet" "~" (at 143.51 90.17 0)
+      (effects (font (size 1.27 1.27)) hide)
+    )
+    (pin "1")
+    (pin "2")
+    (instances
+      (project "BarLight_v1"
+        (path "/e09a2a5b-1bf6-492a-87e7-b4fbc0e9cc1e"
+          (reference "SW1") (unit 1)
+        )
+      )
